Commit message: Fixed bugs

File: catvehicle_ws/src/catvehicle/urdf/catvehicle.xacro (robot description, xacro)
@@ -390,7 +390,7 @@
 	<axis xyz="0 0 1"/>
 	<parent link="camera_link"/>
-	<child link="velodyne_link"/>
-</joint>
-<link name="velodyne_link">
+	<child link="velodyne"/>
+</joint>
+<link name="velodyne">
         <collision>
           <origin xyz="0 0 0" rpy="0 0 0"/>
